File: simple-h/simple-h.sch (KiCad schematic (older format))
At the start: 27 parts, among them J1 Conn_02x04_Odd_Even, J2 CN1, J3 FAN, J4 M1, J5 M2, J6 B+, J7 B-, Q1 BTS7960B, Q2 BTS7960B

Commit message: Ruteo terminado
Parts:
- added MH1, MH2, MH3, MH4: MountingHole, Mounting_Holes:MountingHole_2.2mm_M2_Pad, symbol Mechanical:MountingHole
- added MH5, MH6, MH7, MH8: MountingHole, Mounting_Holes:MountingHole_4.3mm_M4, symbol Mechanical:MountingHole
- D3, D4, D5: footprint digikey-footprints:DO-214AB -> custom_footprint:DO-214AC_custom
- J4, J5, J6, J7: footprint (none) -> custom_footprint:keystone_7693
- Q1, Q2: footprint Package_TO_SOT_SMD:TO-263-7_TabPin8 -> TO_SOT_Packages_SMD:TO-263-7_TabPin8
Connections:
- net labels removed: CN1-1, CN1-2, CN1-3, CN1-4, CN1-5, CN1-6, CN1-7, CN1-8
- wire segments 106 -> 126
