File: simple-h/simple-h.sch (KiCad schematic (older format))
At the start: 35 parts, among them J1 Conn_02x04_Odd_Even, J2 CN1, J3 FAN, J4 M1, J5 M2, J6 B+, J7 B-, Q1 BTS7960B, Q2 BTS7960B

Commit message: Se agregaron los modelos 3D al proyecto
Parts:
- J3: footprint Connectors_Phoenix:PhoenixContact_MC-G_02x3.50mm_Angled -> w_conn_pt-1,5:pt_1,5-2-3,5-h
Changed lines of the file:
@@
 L Connector:Screw_Terminal_01x02 J3
 U 1 1 5BADE6CC
-P 1600 4900
-F 0 "J3" H 1679 4892 50  0000 L CNN
-F 1 "FAN" H 1679 4801 50  0000 L CNN
-F 2 "Connectors_Phoenix:PhoenixContact_MC-G_02x3.50mm_Angled" H 1600 4900 50  0001 C CNN
-F 3 "~" H 1600 4900 50  0001 C CNN
-	1    1600 4900
-	1    0    0    1
+P 1600 4800
+F 0 "J3" H 1679 4792 50  0000 L CNN
+F 1 "FAN" H 1679 4701 50  0000 L CNN
+F 2 "w_conn_pt-1,5:pt_1,5-2-3,5-h" H 1600 4800 50  0001 C CNN
+F 3 "~" H 1600 4800 50  0001 C CNN
+	1    1600 4800
+	1    0    0    -1
 $EndComp
 $Comp
@@
 L Mechanical:Heatsink_Pad HS2
 U 1 1 5BBFE535
-P 4150 5500
-F 0 "HS2" H 4291 5541 50  0000 L CNN
-F 1 "Heatsink_Pad" H 4291 5450 50  0000 L CNN
-F 2 "Heatsinks:Heatsink_AAVID_573300D00010G_TO-263" H 4162 5450 50  0001 C CNN
-F 3 "~" H 4162 5450 50  0001 C CNN
-	1    4150 5500
+P 2150 6650
+F 0 "HS2" H 2291 6691 50  0000 L CNN
+F 1 "Heatsink_Pad" H 2291 6600 50  0000 L CNN
+F 2 "Heatsinks:Heatsink_AAVID_573300D00010G_TO-263" H 2162 6600 50  0001 C CNN
+F 3 "~" H 2162 6600 50  0001 C CNN
+	1    2150 6650
 	1    0    0    -1
 $EndComp
@@
 M2
 Wire Wire Line
-	4150 5600 4150 5800
-Wire Wire Line
-	4150 5800 4450 5800
+	2150 6750 2150 6950
+Wire Wire Line
+	2150 6950 2450 6950
 $Comp
 L Mechanical:Heatsink_Pad HS1
 U 1 1 5BC05653
-P 3300 5500
-F 0 "HS1" H 3441 5541 50  0000 L CNN
-F 1 "Heatsink_Pad" H 3441 5450 50  0000 L CNN
-F 2 "Heatsinks:Heatsink_AAVID_573300D00010G_TO-263" H 3312 5450 50  0001 C CNN
-F 3 "~" H 3312 5450 50  0001 C CNN
-	1    3300 5500
-	1    0    0    -1
-$EndComp
-Wire Wire Line
-	3300 5600 3300 5800
-Wire Wire Line
-	3300 5800 3600 5800
-Text Label 3600 5800 0    50   ~ 0
+P 1300 6650
+F 0 "HS1" H 1441 6691 50  0000 L CNN
+F 1 "Heatsink_Pad" H 1441 6600 50  0000 L CNN
+F 2 "Heatsinks:Heatsink_AAVID_573300D00010G_TO-263" H 1312 6600 50  0001 C CNN
+F 3 "~" H 1312 6600 50  0001 C CNN
+	1    1300 6650
+	1    0    0    -1
+$EndComp
+Wire Wire Line
+	1300 6750 1300 6950
+Wire Wire Line
+	1300 6950 1600 6950
+Text Label 1600 6950 0    50   ~ 0
 M1
-Text Label 4450 5800 0    50   ~ 0
+Text Label 2450 6950 0    50   ~ 0
 M2
 $Comp

Commit message: Se agregaron fiduciales
Parts:
- added F1, F2, F3: Fiducial, Fiducials:Fiducial_1mm_Dia_2mm_Outer, symbol Mechanical:MountingHole
Other:
- note added: "Agujeros"
- note added: "Alimentación Potencia"
- note added: "Conexiones externas"
- note added: "Disipadores"
- note added: "Interfaz"
- note added: "Puentes H"
- note added: "Señalizaciones"

Commit message: Se aplicaron correcciones basadas en revision
Connections:
- wire segments 126 -> 120
Other:
- note added: "Interfaz lógica y\nalimentación de baja potencia"
- note removed: "Conexiones externas"
- note removed: "Interfaz"
- note removed: "Puentes H"
- note removed: "Señalizaciones"
