File: simple-h/simple-h.kicad_pcb (KiCad board)
At the start: 2 copper layers, 57.2 x 63.5 mm, 35 parts, among them J1 Conn_02x04_Odd_Even, J2 CN1, J3 FAN, J4 M1, J5 M2, J6 B+, J7 B-, Q1 BTS7960B, Q2 BTS7960B

Commit message: Se agregaron fiduciales
Parts:
- added F1: Fiducial, Fiducials:Fiducial_1mm_Dia_2mm_Outer, F.Cu at (137.8, 92.0)
- added F2: Fiducial, Fiducials:Fiducial_1mm_Dia_2mm_Outer, F.Cu at (184.1, 89.2)
- added F3: Fiducial, Fiducials:Fiducial_1mm_Dia_2mm_Outer, F.Cu at (172.9, 44.9)
Changed lines of the file:
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@@
     (tracks 196)
     (zones 0)
-    (modules 35)
+    (modules 38)
     (nets 19)
   )
@@
   )
   (layers
-    (0 F.Cu signal hide)
-    (31 B.Cu signal hide)
+    (0 F.Cu signal)
+    (31 B.Cu signal)
     (32 B.Adhes user)
     (33 F.Adhes user)
@@
   )
   (setup
-    (last_trace_width 0.6)
+    (last_trace_width 0.8)
     (user_trace_width 0.6)
     (trace_clearance 0.2)
@@
     (add_net VDD)
   )
+  (module Fiducials:Fiducial_1mm_Dia_2mm_Outer (layer F.Cu)
+    (at 172.89 44.91)
+    (descr "Circular Fiducial, 1mm bare copper top; 2mm keepout (Level A)")
+    (tags marker)
+    (attr virtual)
+    (fp_text reference F3 (at 2.25 0.14) (layer F.SilkS)
+      (effects (font (size 1 1) (thickness 0.15)))
+    )
+    (fp_text value Fiducial (at 0 2) (layer F.Fab) hide
+      (effects (font (size 1 1) (thickness 0.15)))
+    )
+    (fp_circle (center 0 0) (end 1.25 0) (layer F.CrtYd) (width 0.05))
+    (fp_text user %R (at 0 0) (layer F.Fab)
+      (effects (font (size 0.4 0.4) (thickness 0.06)))
+    )
+    (fp_circle (center 0 0) (end 1 0) (layer F.Fab) (width 0.1))
+    (pad ~ smd circle (at 0 0) (size 1 1) (layers F.Cu F.Mask)
+      (solder_mask_margin 0.5) (clearance 0.5))
+  )
+  (module Fiducials:Fiducial_1mm_Dia_2mm_Outer (layer F.Cu)
+    (at 184.14 89.18)
+    (descr "Circular Fiducial, 1mm bare copper top; 2mm keepout (Level A)")
+    (tags marker)
+    (attr virtual)
+    (fp_text reference F2 (at 0 -2) (layer F.SilkS)
+      (effects (font (size 1 1) (thickness 0.15)))
+    )
+    (fp_text value Fiducial (at 0 2) (layer F.Fab) hide
+      (effects (font (size 1 1) (thickness 0.15)))
+    )
+    (fp_circle (center 0 0) (end 1.25 0) (layer F.CrtYd) (width 0.05))
+    (fp_text user %R (at 0 0) (layer F.Fab)
+      (effects (font (size 0.4 0.4) (thickness 0.06)))
+    )
+    (fp_circle (center 0 0) (end 1 0) (layer F.Fab) (width 0.1))
+    (pad ~ smd circle (at 0 0) (size 1 1) (layers F.Cu F.Mask)
+      (solder_mask_margin 0.5) (clearance 0.5))
+  )
+  (module Fiducials:Fiducial_1mm_Dia_2mm_Outer (layer F.Cu)
+    (at 137.8 91.97)
+    (descr "Circular Fiducial, 1mm bare copper top; 2mm keepout (Level A)")
+    (tags marker)
+    (attr virtual)
+    (fp_text reference F1 (at -2.23 -0.9) (layer F.SilkS)
+      (effects (font (size 1 1) (thickness 0.15)))
+    )
+    (fp_text value Fiducial (at 0 2) (layer F.Fab) hide
+      (effects (font (size 1 1) (thickness 0.15)))
+    )
+    (fp_circle (center 0 0) (end 1.25 0) (layer F.CrtYd) (width 0.05))
+    (fp_text user %R (at 0 0) (layer F.Fab)
+      (effects (font (size 0.4 0.4) (thickness 0.06)))
+    )
+    (fp_circle (center 0 0) (end 1 0) (layer F.Fab) (width 0.1))
+    (pad ~ smd circle (at 0 0) (size 1 1) (layers F.Cu F.Mask)
+      (solder_mask_margin 0.5) (clearance 0.5))
+  )
   (module Mounting_Holes:MountingHole_2.2mm_M2_Pad (layer F.Cu)
     (at 134.2 94.2)
@@
     (descr "Through hole straight pin header, 2x04, 2.54mm pitch, double rows")
     (tags "Through hole pin header THT 2x04 2.54mm double row")
-    (fp_text reference J1 (at 1.27 -2.33 90) (layer F.SilkS)
+    (fp_text reference J1 (at 5.01 -0.95 180) (layer F.SilkS)
       (effects (font (size 1 1) (thickness 0.15)))
     )
@@
     (tags "resistor 1206")
     (attr smd)
-    (fp_text reference R1 (at 3.25 -0.5 180) (layer F.SilkS)
-      (effects (font (size 1 1) (thickness 0.15)))
-    )
+    (fp_text reference R1 (at -3.44 0.02 180) (layer F.SilkS)
+      (effects (font (size 1 1) (thickness 0.15)))
+    )

Commit message: Se aplicaron correcciones basadas en revision
Other:
- board text added: "Mínimos (Mayer 10 mils): Grillas: 1mm, 0.5mm Vía: 0.8mm Margen: 0.25mm Pista: 0.6mm, 0.8mm Dist. a borde: 0.3mm"
- board text removed: "Mínimos (Mayer 10 mils): Grillas: 1mm, 0.5mm Vía: 0.8mm Margen: 0.25mm Pista: 0.6mm, 0.8mm Dist. a borde: 0.3mm Terminación: HASL"
Changed lines of the file:
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@@
     )
   )
-  (gr_text "Mínimos (Mayer 10 mils):\nGrillas: 1mm, 0.5mm\nVía: 0.8mm\nMargen: 0.25mm\nPista: 0.6mm, 0.8mm\nDist. a borde: 0.3mm\nTerminación: HASL" (at 206.73 65.1) (layer Dwgs.User)
-    (effects (font (size 1.5 1.5) (thickness 0.3)) (justify left))
+  (gr_text "Mínimos (Mayer 10 mils):\nGrillas: 1mm, 0.5mm\nVía: 0.8mm\nMargen: 0.25mm\nPista: 0.6mm, 0.8mm\nDist. a borde: 0.3mm" (at 206.73 65.1) (layer Dwgs.User)
+    (effects (font (size 1.5 1.5) (thickness 0.1)) (justify left))
   )
-  (dimension 63.5 (width 0.3) (layer Dwgs.User)
+  (dimension 63.5 (width 0.1) (layer Dwgs.User)
     (gr_text "63.500 mm" (at 199.79 65.26 270) (layer Dwgs.User)
-      (effects (font (size 1.5 1.5) (thickness 0.3)))
+      (effects (font (size 1.5 1.5) (thickness 0.1)))
     )
     (feature1 (pts (xy 188.59 97.01) (xy 198.276421 97.01)))
